Commit message: added moveit config, made ball_butler_support an actual ros package. Currently having erros when running moveit demo launch

File: ball_butler_support/urdf/robot.urdf (robot description, URDF)
Before this commit: robot onshape_urdf, 4 links, 3 joints
Links:
- link base: geometry collision mesh filename=package://ball_butler_support/mesh/base.stl; visual mesh filename=package://ball_butler_support/mesh/base.stl
- link hand: geometry collision mesh filename=package://ball_butler_support/mesh/hand.stl; visual mesh filename=package://ball_butler_support/mesh/hand.stl
- link lid: geometry collision mesh filename=package://ball_butler_support/mesh/lid.stl; visual mesh filename=package://ball_butler_support/mesh/lid.stl
- link pitch: geometry collision mesh filename=package://ball_butler_support/mesh/pitch.stl; visual mesh filename=package://ball_butler_support/mesh/pitch.stl
Joints:
- joint pitch: origin xyz=0.041 0.025 -0.0135 rpy=-1.5708 0.771723 7.57459e-16 -> xyz=0.041 0.025 -0.0135 rpy=-1.5708 0.771723 0
- joint throw: origin xyz=-0.01 0.0949984 8.67362e-17 rpy=1.5708 -1.5708 0 -> xyz=-0.01 0.0949984 0 rpy=1.5708 -1.5708 0
- joint yaw: origin xyz=-3.12958e-20 2.12718e-19 0.0565 rpy=3.14159 -0 -3.07134 -> xyz=0 0 0.0565 rpy=3.14159 -0 -3.07134
